File: BigFace.brd (EAGLE design)
At the start: 85.1 x 55.9 mm, 47 parts, among them IC1 MCP23S17SP, IC3 L293E, IC4 L293E, IC5 L293E

Commit message: Updated BRD/SCH
Routing:
- net GND: track 239.4 -> 212.1 mm
Changed lines of the file:
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@@
 <signal name="GND">
 <contactref element="U$1" pad="6"/>
-<contactref element="IC3" pad="4"/>
-<contactref element="IC3" pad="5"/>
-<contactref element="IC5" pad="4"/>
-<contactref element="IC5" pad="5"/>
-<contactref element="IC4" pad="5"/>
-<contactref element="IC4" pad="4"/>
-<contactref element="IC3" pad="13"/>
-<contactref element="IC5" pad="13"/>
-<contactref element="IC5" pad="12"/>
-<contactref element="IC4" pad="13"/>
-<contactref element="IC4" pad="12"/>
-<contactref element="IC3" pad="12"/>
 <contactref element="D5" pad="A"/>
 <contactref element="D8" pad="A"/>
@@
 <wire x1="22.86" y1="6.35" x2="24.13" y2="7.62" width="0.4064" layer="1"/>
 <wire x1="24.13" y1="7.62" x2="24.13" y2="12.7" width="0.4064" layer="1"/>
-<wire x1="36.83" y1="5.08" x2="39.37" y2="5.08" width="0.4064" layer="1"/>
-<wire x1="36.83" y1="12.7" x2="39.37" y2="12.7" width="0.4064" layer="1"/>
-<wire x1="36.83" y1="17.78" x2="39.37" y2="17.78" width="0.4064" layer="1"/>
-<wire x1="36.83" y1="30.48" x2="39.37" y2="30.48" width="0.4064" layer="1"/>
-<wire x1="36.83" y1="38.1" x2="39.37" y2="38.1" width="0.4064" layer="1"/>
 <wire x1="24.13" y1="35.56" x2="24.13" y2="12.7" width="0.4064" layer="1"/>
 <contactref element="IC1" pad="10"/>
@@
 <wire x1="25.4" y1="2.54" x2="36.195" y2="2.54" width="0.4064" layer="1"/>
 <wire x1="36.195" y1="2.54" x2="36.83" y2="3.175" width="0.4064" layer="1"/>
-<wire x1="36.83" y1="3.175" x2="36.83" y2="5.08" width="0.4064" layer="1"/>
 <wire x1="61.595" y1="43.815" x2="62.865" y2="43.815" width="0.4064" layer="16"/>
 <wire x1="62.865" y1="43.815" x2="63.5" y2="44.45" width="0.4064" layer="16"/>
@@
 <wire x1="53.975" y1="53.975" x2="53.975" y2="51.435" width="0.4064" layer="16"/>
 <wire x1="53.975" y1="51.435" x2="53.975" y2="48.895" width="0.4064" layer="16"/>
-<wire x1="39.37" y1="17.78" x2="39.37" y2="25.4" width="0.4064" layer="16"/>
-<wire x1="39.37" y1="30.48" x2="39.37" y2="36.195" width="0.4064" layer="16"/>
-<wire x1="39.37" y1="12.7" x2="39.37" y2="17.78" width="0.4064" layer="1"/>
-<wire x1="36.83" y1="25.4" x2="39.37" y2="25.4" width="0.4064" layer="1"/>
-<wire x1="39.37" y1="25.4" x2="39.37" y2="30.48" width="0.4064" layer="1"/>
-<wire x1="39.37" y1="38.1" x2="39.37" y2="36.195" width="0.4064" layer="16"/>
 <wire x1="39.37" y1="36.195" x2="42.545" y2="36.195" width="0.4064" layer="16"/>
 <wire x1="42.545" y1="36.195" x2="43.18" y2="36.83" width="0.4064" layer="16"/>
@@
 <contactref element="C2" pad="2"/>
 <contactref element="C1" pad="2"/>
-<wire x1="39.37" y1="12.7" x2="39.37" y2="5.08" width="0" layer="19" extent="1-1"/>
 <wire x1="24.13" y1="43.815" x2="27.305" y2="43.815" width="0.4064" layer="16"/>
 <wire x1="27.305" y1="43.815" x2="28.575" y2="42.545" width="0.4064" layer="16"/>
 <wire x1="13.335" y1="8.89" x2="13.335" y2="8.255" width="0.4064" layer="1"/>
 <wire x1="13.335" y1="8.255" x2="16.51" y2="5.08" width="0.4064" layer="1"/>
+<contactref element="IC3" pad="4"/>
+<contactref element="IC3" pad="5"/>
+<contactref element="IC5" pad="4"/>
+<contactref element="IC5" pad="5"/>
+<contactref element="IC4" pad="5"/>
+<contactref element="IC4" pad="4"/>
+<wire x1="36.83" y1="5.08" x2="39.37" y2="5.08" width="0.4064" layer="1"/>
+<wire x1="36.83" y1="17.78" x2="39.37" y2="17.78" width="0.4064" layer="1"/>
+<wire x1="36.83" y1="30.48" x2="39.37" y2="30.48" width="0.4064" layer="1"/>
+<contactref element="IC3" pad="13"/>
+<contactref element="IC5" pad="13"/>
+<contactref element="IC5" pad="12"/>
+<contactref element="IC4" pad="13"/>
+<contactref element="IC4" pad="12"/>
+<contactref element="IC3" pad="12"/>
+<wire x1="36.83" y1="12.7" x2="39.37" y2="12.7" width="0.4064" layer="1"/>
+<wire x1="36.83" y1="38.1" x2="39.37" y2="38.1" width="0.4064" layer="1"/>
+<wire x1="36.83" y1="25.4" x2="39.37" y2="25.4" width="0.4064" layer="1"/>
+<wire x1="39.37" y1="38.1" x2="39.37" y2="36.195" width="0" layer="19" extent="16-16"/>
+<wire x1="39.37" y1="30.48" x2="39.37" y2="36.195" width="0" layer="19" extent="16-16"/>
+<wire x1="39.37" y1="25.4" x2="39.37" y2="30.48" width="0" layer="19" extent="1-1"/>
+<wire x1="39.37" y1="17.78" x2="39.37" y2="25.4" width="0" layer="19" extent="1-1"/>
+<wire x1="39.37" y1="12.7" x2="39.37" y2="17.78" width="0" layer="19" extent="1-1"/>
+<wire x1="39.37" y1="5.08" x2="39.37" y2="12.7" width="0" layer="19" extent="1-1"/>
+<wire x1="36.83" y1="3.175" x2="36.83" y2="5.08" width="0" layer="19" extent="1-1"/>
 </signal>
 <signal name="M1SA">
